File: MONGO_PCB_DESIGN_V2/MONGO_PCB_DESIGN_V2/MONGO_PCB_DESIGN_V2.kicad_pcb (KiCad board)
At the start: 2 copper layers, 117.9 x 56.4 mm, 4 parts

Commit message: PCB modif
Parts:
- removed the REF** at (126.5, 57.9)
- added REF**: TerminalBlock_MaiXu_MX126-5.0-09P_1x09_P5.00mm, TerminalBlock:TerminalBlock_MaiXu_MX126-5.0-09P_1x09_P5.00mm, F.Cu at (203.7, 83.3)
- moved CD74HC4067 79.4 mm to (158.0, 50.8)
- moved CD74HC4067 79.4 mm to (114.8, 50.8)
- moved REF** 79.4 mm to (170.7, 80.0)
Routing:
- net (no net): track 1438.5 -> 1964.1 mm, vias 9 -> 11
Other:
- board outline removed
- board text added: "EN"
- board text added: "GND"
- board text added: "S0"
- board text added: "S1"
- board text added: "S2"
- board text added: "S3"
- board text added: "SIG OUT 1"
- board text added: "SIG OUT 2"
- board text added: "VCC"

Commit message: -
Parts:
- added REF**: PinHeader_1x04_P2.54mm_Vertical, Connector_PinHeader_2.54mm:PinHeader_1x04_P2.54mm_Vertical, F.Cu at (20.3, 111.8)
- added REF**: PinHeader_1x04_P2.54mm_Vertical, Connector_PinHeader_2.54mm:PinHeader_1x04_P2.54mm_Vertical, F.Cu at (20.3, 127.0)
- moved CD74HC4067 124.6 mm to (80.6, 148.5)
- moved CD74HC4067 124.6 mm to (37.4, 148.5)
- moved REF** 124.6 mm to (93.3, 177.7)
- moved REF** 93.2 mm to (111.1, 94.0), turned to 180 degrees
Routing:
- net (no net): track 1964.1 -> 1438.5 mm, vias 11 -> 9
Other:
- board outline added: 100 x 100 mm

Commit message: some work on pcb
Parts:
- removed the REF** at (20.3, 111.8)
- removed the REF** at (20.3, 127.0)
- added CD74HC4067: TensarRobot_CD74HC4067, own:TensarRobot_CD74HC4067, F.Cu at (205.0, 74.2)
- added CD74HC4067: TensarRobot_CD74HC4067, own:TensarRobot_CD74HC4067, F.Cu at (248.2, 74.2)
- added REF**: PinHeader_1x04_P2.54mm_Vertical, Connector_PinHeader_2.54mm:PinHeader_1x04_P2.54mm_Vertical, F.Cu at (187.9, 52.7)
- added REF**: DSUB-15_Pins_Horizontal_P2.77x2.84mm_EdgePinOffset9.90mm_Ho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, Connector_Dsub:DSUB-15_Pins_Horizontal_P2.77x2.84mm_EdgePinOffset9.90mm_Housed_MountingHolesOffset11.32mm, F.Cu at (245.4, 101.6)
- added REF**: HUM.SENSOR.LD, own:Soil_Moisture_Sensor_Module, F.Cu at (30.5, 116.8)
- added REF**: DSUB-9_Pins_Horizontal_P2.77x2.84mm_EdgePinOffset4.94mm_Hou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, Connector_Dsub:DSUB-9_Pins_Horizontal_P2.77x2.84mm_EdgePinOffset4.94mm_Housed_MountingHolesOffset4.94mm, F.Cu at (320.0, 134.6)
- added REF**: HUM.SENSOR.LD, own:Soil_Moisture_Sensor_Module, F.Cu at (30.5, 104.6)
- added REF**: DSUB-15_Pins_Horizontal_P2.77x2.84mm_EdgePinOffset9.90mm_Ho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, Connector_Dsub:DSUB-15_Pins_Horizontal_P2.77x2.84mm_EdgePinOffset9.90mm_Housed_MountingHolesOffset11.32mm, F.Cu at (199.2, 101.6)
- added REF**: TerminalBlock_MaiXu_MX126-5.0-09P_1x09_P5.00mm, TerminalBlock:TerminalBlock_MaiXu_MX126-5.0-09P_1x09_P5.00mm, F.Cu at (278.7, 19.7)
- added REF**: PinHeader_1x04_P2.54mm_Vertical, Connector_PinHeader_2.54mm:PinHeader_1x04_P2.54mm_Vertical, F.Cu at (187.9, 37.5)
- CD74HC4067: value TensarRobot_CD74HC4067 -> Untitled
- moved CD74HC4067 21.7 mm to (57.8, 156.1), turned to 90 degrees
- moved REF** 9.84 mm to (101.3, 94.0)
- moved CD74HC4067 1.81 mm to (81.9, 147.2), turned to 90 degrees
Routing:
- net (no net): track 1438.5 -> 3168.5 mm, vias 9 -> 21
Other:
- board size 100 x 100 mm -> 267.6 x 174.3 mm

Commit message: pcb modfng
Parts:
- removed the CD74HC4067 at (205.0, 74.2)
- removed the CD74HC4067 at (248.2, 74.2)
- removed the REF** at (187.9, 52.7)
- removed the REF** at (245.4, 101.6)
- removed the REF** at (320.0, 134.6)
- removed the REF** at (199.2, 101.6)
- removed the REF** at (278.7, 19.7)
- removed the REF** at (187.9, 37.5)
- CD74HC4067: value TensarRobot_CD74HC4067 -> Untitled
- moved CD74HC4067 21.0 mm to (100.9, 156.1)
Connections:
- CD74HC4067 pad 1: (no net) -> C0-1
- CD74HC4067 pad 10: (no net) -> C9-1
- CD74HC4067 pad 11: (no net) -> C10-1
- CD74HC4067 pad 12: (no net) -> C11-1
- CD74HC4067 pad 13: (no net) -> C12-1
- CD74HC4067 pad 14: (no net) -> C13-1
- CD74HC4067 pad 15: (no net) -> C14-1
- CD74HC4067 pad 16: (no net) -> C15-1
- CD74HC4067 pad 18: (no net) -> GND (x2)
- CD74HC4067 pad 19: (no net) -> VCC (x2)
- CD74HC4067 pad 2: (no net) -> C1-1
- CD74HC4067 pad 20: (no net) -> EN (x2)
- CD74HC4067 pad 21: (no net) -> S0 (x2)
- CD74HC4067 pad 22: (no net) -> S1 (x2)
- CD74HC4067 pad 23: (no net) -> S2 (x2)
- CD74HC4067 pad 24: (no net) -> S3 (x2)
- CD74HC4067 pad 25: (no net) -> SIG-1
- CD74HC4067 pad 3: (no net) -> C2-1
- CD74HC4067 pad 4: (no net) -> C3-1
- CD74HC4067 pad 5: (no net) -> C4-1
- CD74HC4067 pad 6: (no net) -> C5-1
- CD74HC4067 pad 7: (no net) -> C6-1
- CD74HC4067 pad 8: (no net) -> C7-1
- CD74HC4067 pad 9: (no net) -> C8-1
- CD74HC4067 pad 1: (no net) -> C0-2
- CD74HC4067 pad 10: (no net) -> C9-2
- CD74HC4067 pad 11: (no net) -> C10-2
- CD74HC4067 pad 12: (no net) -> C11-2
- CD74HC4067 pad 13: (no net) -> C12-2
- CD74HC4067 pad 14: (no net) -> C13-2
- CD74HC4067 pad 15: (no net) -> C14-2
- CD74HC4067 pad 16: (no net) -> C15-2
- CD74HC4067 pad 2: (no net) -> C1-2
- CD74HC4067 pad 25: (no net) -> SIG-2
- CD74HC4067 pad 3: (no net) -> C2-2
- CD74HC4067 pad 4: (no net) -> C3-2
- CD74HC4067 pad 5: (no net) -> C4-2
- CD74HC4067 pad 6: (no net) -> C5-2
- CD74HC4067 pad 7: (no net) -> C6-2
- CD74HC4067 pad 8: (no net) -> C7-2
- CD74HC4067 pad 9: (no net) -> C8-2
- REF** pad 1: (no net) -> C0-1
- REF** pad 10: (no net) -> C9-1
- REF** pad 11: (no net) -> C10-1
- REF** pad 12: (no net) -> C11-1
- REF** pad 13: (no net) -> C12-1
- REF** pad 14: (no net) -> C13-1
- REF** pad 15: (no net) -> C14-1
- REF** pad 16: (no net) -> C15-1
- REF** pad 2: (no net) -> C1-1
- REF** pad 20: (no net) -> C0-2
- REF** pad 21: (no net) -> C1-2
- REF** pad 22: (no net) -> C2-2
- REF** pad 23: (no net) -> C3-2
- REF** pad 24: (no net) -> C4-2
- REF** pad 25: (no net) -> C5-2
- REF** pad 26: (no net) -> C6-2
- REF** pad 27: (no net) -> C7-2
- REF** pad 28: (no net) -> C8-2
- REF** pad 29: (no net) -> C9-2
- REF** pad 3: (no net) -> C2-1
- REF** pad 30: (no net) -> C10-2
- REF** pad 31: (no net) -> C11-2
- REF** pad 32: (no net) -> C12-2
- REF** pad 33: (no net) -> C13-2
- REF** pad 34: (no net) -> C14-2
- REF** pad 35: (no net) -> C15-2
- REF** pad 4: (no net) -> C3-1
- REF** pad 5: (no net) -> C4-1
- REF** pad 6: (no net) -> C5-1
- REF** pad 7: (no net) -> C6-1
- REF** pad 8: (no net) -> C7-1
- REF** pad 9: (no net) -> C8-1
- REF** pad 1: (no net) -> VCC (x2)
- REF** pad 2: (no net) -> GND (x2)
- REF** pad 4: (no net) -> A0-2
- REF** pad 4: (no net) -> A0-1
- REF** pad 1: (no net) -> GND
- REF** pad 2: (no net) -> VCC
- REF** pad 3: (no net) -> EN
- REF** pad 4: (no net) -> S0
- REF** pad 5: (no net) -> S1
- REF** pad 6: (no net) -> S2
- REF** pad 7: (no net) -> S3
- REF** pad 8: (no net) -> A0-2
- REF** pad 9: (no net) -> A0-1
Routing:
- net (no net): track 3168.5 -> 0.00 mm, vias 21 -> 0
- net GND: track 0.00 -> 201.0 mm, vias 0 -> 1
- net VCC: track 0.00 -> 193.0 mm, vias 0 -> 3
- net EN: track 0.00 -> 96.0 mm, vias 0 -> 2
- net S0: track 0.00 -> 93.9 mm, vias 0 -> 2
- net S3: track 0.00 -> 93.5 mm, vias 0 -> 1
- net S2: track 0.00 -> 93.3 mm
- net S1: track 0.00 -> 92.0 mm, vias 0 -> 2
- net A0-2: track 0.00 -> 62.9 mm
- net A0-1: track 0.00 -> 50.0 mm
- net C0-2: track 0.00 -> 46.6 mm
- net C1-2: track 0.00 -> 46.2 mm
- net C2-2: track 0.00 -> 46.1 mm
- net C3-2: track 0.00 -> 45.7 mm
- net C4-2: track 0.00 -> 45.6 mm
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Other:
- board size 267.6 x 174.3 mm -> 100 x 98 mm
- board text added: "Mongo Garden Connector Module V1"
- board text added: "by: SR211007 © 2026"

Commit message: .
Connections:
- REF** pad 5: (no net) -> GND (x2)
- REF** pad 6: (no net) -> GND (x2)
Routing:
- net GND: track 201.0 -> 263.9 mm
- net SIG-1: track 0.00 -> 52.2 mm
- net SIG-2: track 0.00 -> 34.3 mm
- net A0-2: track 62.9 -> 65.6 mm
- net A0-1: track 50.0 -> 51.5 mm
- net VCC: track 193.0 -> 194.3 mm

Commit message: PCB
Routing:
- net VCC: track 194.3 -> 193.3 mm
- net GND: track 263.9 -> 262.9 mm

Commit message: -
Parts:
- added REF**: TerminalBlock_MaiXu_MX126-5.0-02P_1x02_P5.00mm, TerminalBlock:TerminalBlock_MaiXu_MX126-5.0-02P_1x02_P5.00mm, F.Cu at (109.5, 106.7)
Connections:
- REF** pad 0: (no net) -> GND
- REF** pad 19: (no net) -> GND
- REF** pad 36: (no net) -> RELAY-L
- REF** pad 37: (no net) -> RELAY-R
Routing:
- net RELAY-L: track 0.00 -> 143.1 mm
- net RELAY-R: track 0.00 -> 140.9 mm
- net GND: track 262.9 -> 363.4 mm
Other:
- board text added: "DO NOT USE METAL SCREWS!"
- board text added: "RELAY-L"
- board text added: "RELAY-R"

Commit message: -
Routing:
- net GND: track 363.4 -> 386.1 mm
Changed lines of the file:
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@@
-	)
-	(segment
-		(start 47.5996 140.8684)
-		(end 60.1612 153.43)
-		(width 0.5)
-		(layer "B.Cu")
-		(net 3)
 	)
 	(segment
@@
 	)
 	(segment
-		(start 60.1612 153.43)
-		(end 60.1612 156.7942)
-		(width 0.5)
-		(layer "B.Cu")
-		(net 3)
-	)
-	(segment
 		(start 17.78 104.648)
 		(end 20.32 107.188)
@@
 	)
 	(segment
+		(start 15.9906 158.4056)
+		(end 36.66 179.075)
+		(width 0.5)
+		(layer "B.Cu")
+		(net 3)
+	)
+	(segment
+		(start 15.9906 118.6434)
+		(end 15.9906 158.4056)
+		(width 0.5)
+		(layer "B.Cu")
+		(net 3)
+	)
+	(segment
 		(start 21.8948 100.5332)
 		(end 17.78 104.648)
@@
 	)
 	(segment
-		(start 43.48 173.4754)
-		(end 43.48 177.655)
+		(start 17.794 116.84)
+		(end 15.9906 118.6434)
 		(width 0.5)
 		(layer "B.Cu")
-		(net 3)
-	)
-	(segment
-		(start 60.1612 156.7942)
-		(end 43.48 173.4754)
-		(width 0.5)
-		(layer "B.Cu")
