File: MONGO_PCB_DESIGN_V3/PCB_V3/PCB_V3.kicad_pcb (KiCad board)
At the start: 2 copper layers, 100 x 98 mm, 30 parts, among them Q1 2N2222 TO-92, Q2 2N2222 TO-92, Q3 2N2222 TO-92

Commit message: -
Parts:
- removed the SENSOR MODULE at (58.4, 16.5)
- added G***: LOGO, LOGO, F.Cu at (72.9, 32.4)
- added SENSOR MODULE: JST_PH_B10B-PH-K_1x10_P2.00mm_Vertical, Connector_JST:JST_PH_B10B-PH-K_1x10_P2.00mm_Vertical, F.Cu at (56.0, 16.5)
Other:
- board text added: "RETURN PROBE SIG OUT 2 SIG OUT 1 S3 S2 S1 S0 EN VCC GND"
- board text removed: "SIG OUT 2 SIG OUT 1 S3 S2 S1 S0 EN VCC GND"

Commit message: -
Parts:
- moved G*** 3.32 mm to (71.9, 35.6)
- moved R5 100Ω 0.12 mm to (72.9, 90.1)
Connections:
- 2N7002 pad 3: (no net) -> GATE_AO3401A_PULLUP
- D1 1N4004 pad 1: (no net) -> 5V
- D1 1N4004 pad 2: (no net) -> Q1-D1
- D2 1N4004 pad 1: (no net) -> 5V
- D2 1N4004 pad 2: (no net) -> Q2-D2
- D3 1N4004 pad 1: (no net) -> 5V
- D3 1N4004 pad 2: (no net) -> Q3-D3
- Q1 2N2222 pad 2: (no net) -> R1-Q1
- Q1 2N2222 pad 3: (no net) -> Q1-D1
- Q2 2N2222 pad 2: (no net) -> R2-Q2
- Q2 2N2222 pad 3: (no net) -> Q2-D2
- Q3 2N2222 pad 2: (no net) -> R3-Q3
- Q3 2N2222 pad 3: (no net) -> Q3-D3
- R1 1KΩ pad 2: (no net) -> R1-Q1
- R2 1KΩ pad 2: (no net) -> R2-Q2
- R3 1KΩ pad 2: (no net) -> R3-Q3
- R5 100Ω pad 1: (no net) -> GATE_2N7002_PULLDOWN
- REF** pad 10: (no net) -> SDA
- REF** pad 12: (no net) -> SDA
- REF** pad 16: (no net) -> SCL
- REF** pad 18: (no net) -> SCL
- REF** pad 20: (no net) -> SCL
- REF** pad 8: (no net) -> SDA
- RLY1 pad 2: (no net) -> Q1-D1
- RLY2 pad 2: (no net) -> Q2-D2
- RLY3 pad 2: (no net) -> Q3-D3
- SENSOR MODULE pad 1: (no net) -> GPIO35
Routing:
- net (no net): track 68.6 -> 0.00 mm
- net GPIO35: track 68.9 -> 108.3 mm
- net Q3-D3: track 0.00 -> 17.9 mm
- net Q1-D1: track 0.00 -> 17.9 mm
- net Q2-D2: track 0.00 -> 17.9 mm
- net GPIO38: track 64.9 -> 71.1 mm
- net R1-Q1: track 0.00 -> 4.93 mm
- net R2-Q2: track 0.00 -> 4.93 mm
- net R3-Q3: track 0.00 -> 4.93 mm
- net VCC_CONECTOR_MODULE: track 67.9 -> 63.7 mm
- net GPIO40: track 95.8 -> 99.4 mm
- net GPIO45: track 117.6 -> 121.3 mm
- net GPIO41: track 101.2 -> 104.8 mm
- net GPIO42: track 111.3 -> 114.9 mm
- net GPIO48: track 131.1 -> 134.5 mm
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- added copper zone on F.Cu, net GND
