File: MONGO_PCB_DESIGN_V3/PCB_V3/PCB_V3.kicad_pcb (KiCad board)
At the start: 2 copper layers, 100 x 98 mm, 31 parts, among them Q1 2N2222 TO-92, Q2 2N2222 TO-92, Q3 2N2222 TO-92

Commit message: -
Parts:
- moved G*** 240.3 mm to (312.2, 32.5)
Changed lines of the file:
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@@
 	(footprint "LOGO"
 		(layer "F.Cu")
-		(at 71.866609 35.582821)
+		(at 312.181771 32.535723)
 		(property "Reference" "G***"
 			(at 0 0 0)

Commit message: -
Parts:
- removed SD CARD MODULE: mini TF card, own:mini TF card
- added G***: LOGO, LOGO, B.Cu at (62.7, 61.0)
- added TF card: MICROSD, own:MICROSD, F.Cu at (17.0, 53.0)
- I2C-1: renamed from Generic I2C-1
- I2C-2: renamed from Generic I2C-2
- I2C-3: renamed from Generic I2C-3
- moved G*** 241.2 mm to (71.0, 34.0)
- renumbered TSL2561 to I2C-4, BMP180-int to I2C-5, BMP180-ext to I2C-6
Connections:
- REF** pad 7: GPIO36 -> SIG_BATTERY
- REF** pad 36: GPIO36 -> SIG_BATTERY
Routing:
- net SIG_BATTERY: track 0.00 -> 138.3 mm, vias 0 -> 3
- net GPIO36: track 68.6 -> 0.00 mm, vias 1 -> 0
- net CS: track 29.6 -> 19.3 mm
- net MISO: track 17.9 -> 24.3 mm, vias 0 -> 2
- net 5V_RAIL: track 151.7 -> 155.2 mm
- net MOSI: track 21.0 -> 18.2 mm
- net 12V: track 195.4 -> 192.8 mm
- net 5V: track 348.0 -> 350.5 mm
- net SCK: track 23.1 -> 20.9 mm, vias 0 -> 2
- net TX: track 96.5 -> 97.1 mm

Commit message: -
Connections:
- REF** pad 21: ENABLE_RLY1 -> GPIO48
- REF** pad 33: ENABLE_RLY2 -> GPIO47
- REF** pad 34: ENABLE_RLY3 -> GPIO45
- REF** pad 35: GPIO35 -> GPIO42
- REF** pad 36: SIG_BATTERY -> GPIO41
- REF** pad 37: GPIO37 -> GPIO40
- REF** pad 38: GPIO38 -> GPIO39
- REF** pad 39: GPIO39 -> GPIO38
- REF** pad 40: GPIO40 -> GPIO37
- REF** pad 41: GPIO41 -> SIG_BATTERY
- REF** pad 42: GPIO42 -> GPIO35
- REF** pad 45: GPIO45 -> ENABLE_RLY3
- REF** pad 47: GPIO47 -> ENABLE_RLY2
- REF** pad 48: GPIO48 -> ENABLE_RLY1
Changed lines of the file:
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@@
 		)
 		(pad "21" smd circle
+			(at 3.523012 6.187588)
+			(size 1.5 1.5)
+			(layers "F.Cu" "F.Mask" "F.Paste")
+			(net 12 "GPIO48")
+		)
+		(pad "33" smd circle
+			(at 3.523012 8.347588)
+			(size 1.5 1.5)
+			(layers "F.Cu" "F.Mask" "F.Paste")
+			(net 42 "GPIO47")
+		)
+		(pad "34" smd circle
+			(at 3.523012 10.507588)
+			(size 1.5 1.5)
+			(layers "F.Cu" "F.Mask" "F.Paste")
+			(net 41 "GPIO45")
+		)
+		(pad "35" smd circle
+			(at 3.523012 12.667588)
+			(size 1.5 1.5)
+			(layers "F.Cu" "F.Mask" "F.Paste")
+			(net 40 "GPIO42")
+		)
+		(pad "36" smd circle
+			(at 3.523012 14.827588)
+			(size 1.5 1.5)
+			(layers "F.Cu" "F.Mask" "F.Paste")
+			(net 39 "GPIO41")
+		)
+		(pad "37" smd circle
+			(at 3.523012 16.987588)
+			(size 1.5 1.5)
+			(layers "F.Cu" "F.Mask" "F.Paste")
+			(net 38 "GPIO40")
+		)
+		(pad "38" smd circle
+			(at 3.523012 19.147588)
+			(size 1.5 1.5)
+			(layers "F.Cu" "F.Mask" "F.Paste")
+			(net 37 "GPIO39")
+		)
+		(pad "39" smd circle
+			(at 14.173012 19.147588)
+			(size 1.5 1.5)
+			(layers "F.Cu" "F.Mask" "F.Paste")
+			(net 36 "GPIO38")
+		)
+		(pad "40" smd circle
+			(at 14.173012 16.987588)
+			(size 1.5 1.5)
+			(layers "F.Cu" "F.Mask" "F.Paste")
+			(net 35 "GPIO37")
+		)
+		(pad "41" smd circle
+			(at 14.173012 14.827588)
+			(size 1.5 1.5)
+			(layers "F.Cu" "F.Mask" "F.Paste")
+			(net 15 "SIG_BATTERY")
+		)
+		(pad "42" smd circle
+			(at 14.173012 12.667588)
+			(size 1.5 1.5)
+			(layers "F.Cu" "F.Mask" "F.Paste")
+			(net 34 "GPIO35")
+		)
+		(pad "45" smd circle
+			(at 14.173012 10.507588)
+			(size 1.5 1.5)
+			(layers "F.Cu" "F.Mask" "F.Paste")
+			(net 31 "ENABLE_RLY3")
+		)
+		(pad "47" smd circle
+			(at 14.173012 8.347588)
+			(size 1.5 1.5)
+			(layers "F.Cu" "F.Mask" "F.Paste")
+			(net 29 "ENABLE_RLY2")
+		)
+		(pad "48" smd circle
 			(at 14.173012 6.187588)
 			(size 1.5 1.5)
@@
 			(net 30 "ENABLE_RLY1")
 		)
-		(pad "33" smd circle
-			(at 14.173012 8.347588)
-			(size 1.5 1.5)
-			(layers "F.Cu" "F.Mask" "F.Paste")
-			(net 29 "ENABLE_RLY2")
-		)
-		(pad "34" smd circle
-			(at 14.173012 10.507588)
-			(size 1.5 1.5)
-			(layers "F.Cu" "F.Mask" "F.Paste")
-			(net 31 "ENABLE_RLY3")
-		)
-		(pad "35" smd circle
-			(at 14.173012 12.667588)
-			(size 1.5 1.5)
-			(layers "F.Cu" "F.Mask" "F.Paste")
-			(net 34 "GPIO35")
-		)
-		(pad "36" smd circle
-			(at 14.173012 14.827588)
-			(size 1.5 1.5)
-			(layers "F.Cu" "F.Mask" "F.Paste")
-			(net 15 "SIG_BATTERY")
-		)
-		(pad "37" smd circle
-			(at 14.173012 16.987588)
-			(size 1.5 1.5)
-			(layers "F.Cu" "F.Mask" "F.Paste")
-			(net 35 "GPIO37")
-		)
-		(pad "38" smd circle
-			(at 14.173012 19.147588)
-			(size 1.5 1.5)
-			(layers "F.Cu" "F.Mask" "F.Paste")
-			(net 36 "GPIO38")
-		)
-		(pad "39" smd circle
-			(at 3.523012 19.147588)
-			(size 1.5 1.5)
-			(layers "F.Cu" "F.Mask" "F.Paste")
-			(net 37 "GPIO39")
-		)
-		(pad "40" smd circle
-			(at 3.523012 16.987588)
-			(size 1.5 1.5)
-			(layers "F.Cu" "F.Mask" "F.Paste")
-			(net 38 "GPIO40")
-		)
-		(pad "41" smd circle
-			(at 3.523012 14.827588)
-			(size 1.5 1.5)
-			(layers "F.Cu" "F.Mask" "F.Paste")
-			(net 39 "GPIO41")
-		)
-		(pad "42" smd circle
-			(at 3.523012 12.667588)
-			(size 1.5 1.5)
-			(layers "F.Cu" "F.Mask" "F.Paste")
-			(net 40 "GPIO42")
-		)
-		(pad "45" smd circle
-			(at 3.523012 10.507588)
-			(size 1.5 1.5)
-			(layers "F.Cu" "F.Mask" "F.Paste")
-			(net 41 "GPIO45")
-		)
-		(pad "47" smd circle
-			(at 3.523012 8.347588)
-			(size 1.5 1.5)
-			(layers "F.Cu" "F.Mask" "F.Paste")
-			(net 42 "GPIO47")
-		)
-		(pad "48" smd circle
-			(at 3.523012 6.187588)
-			(size 1.5 1.5)
-			(layers "F.Cu" "F.Mask" "F.Paste")
-			(net 12 "GPIO48")
-		)
 		(pad "GND" smd roundrect
